Commit message: This is initial commit!

File: manipulability/src/schunk.urdf (robot description, URDF)
Before this commit: robot None, 0 links, 0 joints
Links:
- added link arm_1_link, mass 0.01; collision mesh filename=package://erl_lwa4d/meshes/lwa4d/arm_1_link.stl; visual mesh filename=package://erl_lwa4d/meshes/lwa4d/arm_1_link.stl
- added link arm_2_link, mass 0.01; collision mesh filename=package://erl_lwa4d/meshes/lwa4d/arm_2_link_collision.stl; visual mesh filename=package://erl_lwa4d/meshes/lwa4d/arm_2_link.stl
- added link arm_3_link, mass 0.01; collision mesh filename=package://erl_lwa4d/meshes/lwa4d/arm_3_link_collision.stl; visual mesh filename=package://erl_lwa4d/meshes/lwa4d/arm_3_link.stl
- added link arm_4_link, mass 0.01; collision mesh filename=package://erl_lwa4d/meshes/lwa4d/arm_4_link_collision.stl; visual mesh filename=package://erl_lwa4d/meshes/lwa4d/arm_4_link.stl
- added link arm_5_link, mass 0.01; collision mesh filename=package://erl_lwa4d/meshes/lwa4d/arm_5_link_collision.stl; visual mesh filename=package://erl_lwa4d/meshes/lwa4d/arm_5_link.stl
- added link arm_6_link, mass 0.01; collision mesh filename=package://erl_lwa4d/meshes/lwa4d/arm_6_link_collision.stl; visual mesh filename=package://erl_lwa4d/meshes/lwa4d/arm_6_link.stl
- added link arm_7_link, mass 0.01; collision mesh filename=package://erl_lwa4d/meshes/lwa4d/arm_7_link.stl; visual mesh filename=package://erl_lwa4d/meshes/lwa4d/arm_7_link.stl
- added link arm_base_link, mass 0.01
- added link arm_ee_link, mass 0.01
- added link arm_podest_link, mass 0.01; collision mesh filename=package://erl_lwa4d/meshes/lwa4d/arm_podest_link.stl; visual mesh filename=package://erl_lwa4d/meshes/lwa4d/arm_podest_link.stl
- added link world
Joints:
- added joint arm_1_joint: type revolute, parent arm_base_link, child arm_1_link, origin xyz=0 0 0 rpy=0 0 0, axis 0 0 -1, limit lower=-3.12159265359 upper=3.12159265359 effort=216 velocity=0.43633
- added joint arm_2_joint: type revolute, parent arm_1_link, child arm_2_link, origin xyz=0 0 0.240 rpy=-1.57079632679 -1.57079632679 0, axis 0 0 -1, limit lower=-2.12 upper=2.12 effort=216 velocity=0.43633
- added joint arm_3_joint: type revolute, parent arm_2_link, child arm_3_link, origin xyz=0 0 0 rpy=1.57079632679 0 1.57079632679, axis 0 0 -1, limit lower=-3.12159265359 upper=3.12159265359 effort=81.5 velocity=0.4189
- added joint arm_4_joint: type revolute, parent arm_3_link, child arm_4_link, origin xyz=0 0 0.328 rpy=-1.57079632679 -1.57079632679 0, axis 0 0 -1, limit lower=-2.16 upper=2.16 effort=81.5 velocity=0.4189
- added joint arm_5_joint: type revolute, parent arm_4_link, child arm_5_link, origin xyz=0 0 0 rpy=1.57079632679 0 1.57079632679, axis 0 0 -1, limit lower=-3.12159265359 upper=3.12159265359 effort=20.7 velocity=0.43633
- added joint arm_6_joint: type revolute, parent arm_5_link, child arm_6_link, origin xyz=0 0 0.323 rpy=-1.57079632679 -1.57079632679 0, axis 0 0 -1, limit lower=-2.07 upper=2.07 effort=15 velocity=1.2566
- added joint arm_7_joint: type revolute, parent arm_6_link, child arm_7_link, origin xyz=0 0 0 rpy=1.57079632679 0 1.57079632679, axis 0 0 -1, limit lower=-2.94 upper=2.94 effort=15 velocity=1.2566
- added joint arm_base_joint: type fixed, parent arm_podest_link, child arm_base_link, origin xyz=0 0 0.140 rpy=0 0 0
- added joint arm_ee_joint: type fixed, parent arm_7_link, child arm_ee_link, origin xyz=0 0 0.0824 rpy=0 0 0
- added joint arm_podest_joint: type fixed, parent world, child arm_podest_link, origin xyz=0 0 0 rpy=0 0 0
